Commit message: 0322

File: sim_car/car_description/robot/car.urdf.xacro (robot description, xacro)
@@ -15,15 +15,15 @@
   <xacro:property name="chassis_mass" value = "${total_mass-4*wheel_mass}"/>
   <xacro:macro name="cylinder_inertia" params="m r h">
-        <inertia  ixx="${m*(3*r*r+h*h)/12}" ixy = "0" ixz = "0"
+    <inertia  ixx="${m*(3*r*r+h*h)/12}" ixy = "0" ixz = "0"
                     iyy="${m*(3*r*r+h*h)/12}" iyz = "0"
                     izz="${m*r*r/2}" />
   </xacro:macro>
   <xacro:macro name="box_inertia" params="m x y z">
-          <inertia  ixx="${m*(y*y+z*z)/12}" ixy = "0" ixz = "0"
+    <inertia  ixx="${m*(y*y+z*z)/12}" ixy = "0" ixz = "0"
                     iyy="${m*(x*x+z*z)/12}" iyz = "0"
                     izz="${m*(x*x+z*z)/12}" />
   </xacro:macro>
   <xacro:macro name="sphere_inertia" params="m r">
-          <inertia  ixx="${2*m*r*r/5}" ixy = "0" ixz = "0"
+    <inertia  ixx="${2*m*r*r/5}" ixy = "0" ixz = "0"
                     iyy="${2*m*r*r/5}" iyz = "0"
                     izz="${2*m*r*r/5}" />
@@ -36,6 +36,5 @@
   </xacro:macro>
   <link name="base_footprint"/>
-  <link name="base_link"/>
-<!--
+  <!-- <link name="base_link"/> -->
   <link name="base_link">
     <visual>
@@ -60,5 +59,4 @@
     </inertial>
   </link>
--->
   <link name="chassis_link">
     <visual>
@@ -114,22 +112,22 @@
   <gazebo reference="laser_scanner_link">
     <sensor type="ray" name="laser_scanner">
-    <always_on>true</always_on>
-    <!-- <visualize>true</visualize> -->
-    <update_rate>3</update_rate>
-    <ray>
-      <scan>
-        <horizontal>
-          <samples>360</samples>
-          <resolution>1</resolution>
-          <min_angle>${-pi}</min_angle>
-          <max_angle>${pi}</max_angle>
-        </horizontal>
-      </scan>
-      <range>
-        <min>0.30</min>
-        <max>25.0</max>
-        <resolution>0.1</resolution>
-      </range>
-    </ray>
+      <always_on>true</always_on>
+      <!-- <visualize>true</visualize> -->
+      <update_rate>3</update_rate>
+      <ray>
+        <scan>
+          <horizontal>
+            <samples>360</samples>
+            <resolution>1</resolution>
+            <min_angle>${-pi}</min_angle>
+            <max_angle>${pi}</max_angle>
+          </horizontal>
+        </scan>
+        <range>
+          <min>0.30</min>
+          <max>25.0</max>
+          <resolution>0.1</resolution>
+        </range>
+      </ray>
       <plugin name="scan" filename="libgazebo_ros_ray_sensor.so">
         <ros>
@@ -177,5 +175,5 @@
     </inertial>
   </link>
-    <link name="front_left_wheel">
+  <link name="front_left_wheel">
     <visual>
       <geometry>
@@ -230,5 +228,5 @@
   </link>
   <link name="back_left_wheel_shock">
-      <visual>
+    <visual>
       <origin xyz="0 0 0.1" rpy="0 0 0"/>
       <geometry>
@@ -253,26 +251,4 @@
   <link name="back_right_wheel_shock">
     <visual>
-    <origin xyz="0 0 0.1" rpy="0 0 0"/>
-    <geometry>
-      <cylinder length="0.05" radius="0.01"/>
-    </geometry>
-    <material name="silver">
-      <color rgba="0.75 0.75 0.75 1"/>
-    </material>
-  </visual>
-  <collision>
-    <origin xyz="0 0 0.1" rpy="0 0 0"/>
-    <geometry>
-      <cylinder length="0.05" radius="0.01"/>
-    </geometry>
-  </collision>
-  <inertial>
-    <mass value="0.01"/>
-    <inertia ixx="0.015" iyy="0.0375" izz="0.0375"
-              ixy="0" ixz="0" iyz="0"/>
-  </inertial>
-</link>
-  <link name="front_left_wheel_shock">
-      <visual>
       <origin xyz="0 0 0.1" rpy="0 0 0"/>
       <geometry>
@@ -292,9 +268,9 @@
       <mass value="0.01"/>
       <inertia ixx="0.015" iyy="0.0375" izz="0.0375"
-               ixy="0" ixz="0" iyz="0"/>
-    </inertial>
-  </link>
-  <link name="front_right_wheel_shock">
-      <visual>
+              ixy="0" ixz="0" iyz="0"/>
+    </inertial>
+  </link>
+  <link name="front_left_wheel_shock">
+    <visual>
       <origin xyz="0 0 0.1" rpy="0 0 0"/>
       <geometry>
@@ -317,10 +293,32 @@
     </inertial>
   </link>
+  <link name="front_right_wheel_shock">
+    <visual>
+      <origin xyz="0 0 0.1" rpy="0 0 0"/>
+      <geometry>
+        <cylinder length="0.05" radius="0.01"/>
+      </geometry>
+      <material name="silver">
+        <color rgba="0.75 0.75 0.75 1"/>
+      </material>
+    </visual>
+    <collision>
+      <origin xyz="0 0 0.1" rpy="0 0 0"/>
+      <geometry>
+        <cylinder length="0.05" radius="0.01"/>
+      </geometry>
+    </collision>
+    <inertial>
+      <mass value="0.01"/>
+      <inertia ixx="0.015" iyy="0.0375" izz="0.0375"
+               ixy="0" ixz="0" iyz="0"/>
+    </inertial>
+  </link>
   <joint name="base_link_joint" type="fixed">
-     <parent link="base_footprint"/>
-     <child link="base_link"/>
-     <origin rpy="0 0 0" xyz="0 0 0"/>
-   </joint>
-   <joint name="laser_scanner_joint" type="fixed">
+    <parent link="base_footprint"/>
+    <child link="base_link"/>
+    <origin rpy="0 0 0" xyz="0 0 0"/>
+  </joint>
+  <joint name="laser_scanner_joint" type="fixed">
     <origin rpy="0 0 0" xyz="0.1397 0 0.2159"/>
     <parent link="base_link"/>
